Commit message: fix: align FS150 viewer assets with Gazebo

File: urdf/fs150_visual.urdf (robot description, URDF)
Before this commit: robot fs150, 6 links, 5 joints
Links:
- link rotor_0: geometry visual mesh filename=package://fs150_description/meshes/iris_prop_ccw.stl scale=1 1 1
- link rotor_1: geometry visual mesh filename=package://fs150_description/meshes/iris_prop_ccw.stl scale=1 1 1
- link rotor_2: geometry visual mesh filename=package://fs150_description/meshes/iris_prop_cw.stl scale=1 1 1
- link rotor_3: geometry visual mesh filename=package://fs150_description/meshes/iris_prop_cw.stl scale=1 1 1
